File: hardware/kicad/simon3/simon3.kicad_sch (KiCad schematic)
At the start: 21 parts, among them J1 Power, J2 Digital/PWM, J3 Analog, J4 Digital/PWM, SW1 SW_Push, SW2 SW_Push, SW3 SW_Push, SW4 SW_Push

Commit message: Ajout clours simon.svg
Other:
- note removed: "* Indicates a PWM-capable pin"
Changed lines of the file:
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@@
-		)
-	)
-	(text "* Indicates a PWM-capable pin"
-		(exclude_from_sim no)
-		(at 177.8 180.34 0)
-		(effects
-			(font
-				(size 1.27 1.27)
-			)
-			(justify left bottom)
 		)
 	)
